File: dcpunks31/dcpunks31.kicad_sch (KiCad schematic)
At the start: 31 parts, among them SW1 SW_SPDT, U1 74HC164, U2 LM556, U3 74HC164, U4 L7805

Commit message: should be ready for mass production
Parts:
- added R3, R4: 1k, Resistor_SMD:R_0603_1608Metric_Pad0.98x0.95mm_HandSolder, symbol Device:R
- BT1: value Battery_Cell -> 9VOLT
- C1, C2: value CP_Small -> 4.7uF; footprint Capacitor_SMD:CP_Elec_8x5.4 -> Capacitor_SMD:CP_Elec_4x5.4
- F1: value Polyfuse -> POLYFUSE; footprint Fuse:Fuse_Bourns_MF-RG400 -> Fuse:Fuse_1206_3216Metric_Pad1.42x1.75mm_HandSolder
- MOD_CLK1: renamed from RV2; value R_POT -> 10k
- MOD_DATA1: renamed from RV1; value R_POT -> 10k
- R1, R2: value R -> 10k; footprint Resistor_SMD:R_0805_2012Metric_Pad1.20x1.40mm_HandSolder -> Resistor_SMD:R_0603_1608Metric_Pad0.98x0.95mm_HandSolder
- RN1, RN2: value R_Pack08 -> RES_PACK
Connections:
- net +5V: now also R3.1, R4.1; no longer MOD_CLK1.1, MOD_DATA1.1
- new net: MOD_CLK1.1, R3.2
- new net: MOD_DATA1.1, R4.2
Other:
- moved on the sheet: C2, MOD_CLK1, R2
