File: dcpunks31/dcpunks31.kicad_pcb (KiCad board)
At the start: 2 copper layers, 91.6 x 99.2 mm, 32 parts, among them SW1 SW_SPDT, U1 74HC164, U2 LM556, U3 74HC164, U4 L7805

Commit message: should be ready for mass production
Parts:
- added R3: 1k, Resistor_SMD:R_0603_1608Metric_Pad0.98x0.95mm_HandSolder, B.Cu at (125.2, 66.7)
- added R4: 1k, Resistor_SMD:R_0603_1608Metric_Pad0.98x0.95mm_HandSolder, B.Cu at (158.2, 68.5)
- BT1: value Battery_Cell -> 9VOLT; moved to B.Cu
- C1, C2: value CP_Small -> 4.7uF; footprint Capacitor_SMD:CP_Elec_8x5.4 -> Capacitor_SMD:CP_Elec_4x5.4
- F1: value Polyfuse -> POLYFUSE; footprint Fuse:Fuse_Bourns_MF-RG400 -> Fuse:Fuse_1206_3216Metric_Pad1.42x1.75mm_HandSolder
- MOD_CLK1: renamed from RV2; value R_POT -> 10k
- MOD_DATA1: renamed from RV1; value R_POT -> 10k
- R1, R2: value R -> 10k; footprint Resistor_SMD:R_0805_2012Metric_Pad1.20x1.40mm_HandSolder -> Resistor_SMD:R_0603_1608Metric_Pad0.98x0.95mm_HandSolder
- RN1, RN2: value R_Pack08 -> RES_PACK
- moved F1 1.96 mm to (171.8, 116.8)
Connections:
- MOD_CLK1 pad 1: +5V -> Net-(MOD_CLK1-Pad1)
- MOD_DATA1 pad 1: +5V -> Net-(MOD_DATA1-Pad1)
Routing:
- net +5V: track 628.8 -> 672.1 mm
- net Net-(MOD_DATA1-Pad1): track 0.00 -> 11.5 mm
- net Net-(MOD_CLK1-Pad1): track 0.00 -> 4.66 mm
- net +9V: track 9.57 -> 8.14 mm
- net Net-(F1-Pad1): track 7.98 -> 7.21 mm
- net Net-(D5-Pad1): track 30.9 -> 31.4 mm
- net /TT_CLK: track 23.5 -> 23.0 mm
- net GND: vias 29 -> 31
Other:
- board text added: "5V_REG"
- board text added: "DUAL_TIMERS"
- board text added: "SHIFT_REG1"
- board text added: "SHIFT_REG2"

Commit message: moar
Parts:
- added G***: LOGO, dcpunks31:logo, B.Cu at (152.1, 93.4)
Routing:
- net GND: vias 31 -> 32
Other:
- board text added: "@kay_kidoutai"
- board text added: "I am so fucking tired of Elon Musk"
- board text added: "SERIAL"
- board text added: "defcon31 2023"
- board text added: "we got no names no names man! we're nameless!"

Commit message: almost done
Parts:
- added G***: LOGO, dcpunks31:htp, B.Cu at (154.7, 98.5)
- added G***: LOGO, dcpunks31:dfiu, B.Cu at (106.9, 91.0)
- moved G*** 7.87 mm to (153.7, 85.7)
Other:
- board text added: "If making money was the point I'd have sold my soul to Raytheon"
- board text added: "MICRO$OFT SUCKS"

Commit message: ordered
Routing:
- net +5V: track 672.1 -> 663.0 mm, vias 4 -> 3
- net Net-(D9-Pad1): track 50.7 -> 52.2 mm
Other:
- board text added: "GET BENT"
- board text added: "I am so fucking tired of Elon Musk [banned for harassment]"
- board text removed: "I am so fucking tired of Elon Musk"
Changed lines of the file:
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@@
   (gr_line (start 134.84 53.65) (end 135.44 54.32) (layer "Edge.Cuts") (width 0.1))
   (gr_line (start 122.23 58.21) (end 117.85 60.82) (layer "Edge.Cuts") (width 0.1))
-  (gr_text "SHIFT_REG2" (at 120.76 85.63) (layer "B.SilkS")
+  (gr_text "SHIFT_REG2" (at 119 86) (layer "B.SilkS")
     (effects (font (size 1.5 1.5) (thickness 0.3)) (justify mirror))
   )
@@
     (effects (font (size 1.5 1.5) (thickness 0.3)) (justify mirror))
   )
+  (gr_text "GET BENT" (at 114 71 15) (layer "B.SilkS")
+    (effects (font (size 1.5 1.5) (thickness 0.3)) (justify mirror))
+  )
   (gr_text "defcon31\n  2023" (at 127.12 138.77) (layer "B.SilkS")
     (effects (font (size 1.5 1.5) (thickness 0.3)) (justify mirror))
   )
-  (gr_text "If making money was the \npoint I'd have sold my\nsoul to Raytheon" (at 137.8 114.74) (layer "B.SilkS")
-    (effects (font (size 1 1) (thickness 0.15)) (justify mirror))
-  )
-  (gr_text "SHIFT_REG1" (at 177.03 87.02) (layer "B.SilkS")
-    (effects (font (size 1.5 1.5) (thickness 0.3)) (justify mirror))
-  )
-  (gr_text "I am so fucking tired\nof Elon Musk" (at 135.7 124.96) (layer "B.Mask")
+  (gr_text "If making money was the \npoint I'd have sold my\nsoul to Raytheon" (at 115 116 90) (layer "B.SilkS")
+    (effects (font (size 1 1) (thickness 0.25)) (justify mirror))
+  )
+  (gr_text "SHIFT_REG1" (at 177 88) (layer "B.SilkS")
+    (effects (font (size 1.5 1.5) (thickness 0.3)) (justify mirror))
+  )
+  (gr_text "I am so fucking tired\nof Elon Musk\n[banned for harassment]" (at 135.5 125) (layer "B.Mask")
     (effects (font (size 1.5 1.5) (thickness 0.3)) (justify mirror))
   )
@@
   (segment (start 122.76 82.91) (end 124.088947 82.91) (width 0.25) (layer "F.Cu") (net 5))
   (segment (start 115.545 129.63) (end 158.44 129.63) (width 0.5) (layer "F.Cu") (net 5))
-  (segment (start 150.65 64.53) (end 150.65 59.85) (width 0.5) (layer "F.Cu") (net 5))
   (segment (start 132.3525 76.0725) (end 133.495 74.93) (width 0.5) (layer "F.Cu") (net 5))
   (segment (start 130.27 78.29) (end 130.27 78.155) (width 0.25) (layer "F.Cu") (net 5))
   (segment (start 166.82 62.29) (end 182.1 77.57) (width 0.5) (layer "F.Cu") (net 5))
-  (segment (start 150.65 59.85) (end 150.59 59.79) (width 0.5) (layer "F.Cu") (net 5))
   (segment (start 125.515 82.91) (end 122.76 82.91) (width 0.5) (layer "F.Cu") (net 5))
   (segment (start 161.895 62.29) (end 166.82 62.29) (width 0.5) (layer "F.Cu") (net 5))
@@
   (via (at 129.89 72.4) (size 0.8) (drill 0.4) (layers "F.Cu" "B.Cu") (net 5))
   (via (at 182.1 78.63) (size 0.8) (drill 0.4) (layers "F.Cu" "B.Cu") (net 5))
-  (via (at 150.65 64.53) (size 0.8) (drill 0.4) (layers "F.Cu" "B.Cu") (net 5))
   (segment (start 158.005 60.94) (end 158.005 67.4225) (width 0.5) (layer "B.Cu") (net 5))
   (segment (start 171.735 110.575) (end 173.85 112.69) (width 0.5) (layer "B.Cu") (net 5))
@@
   (segment (start 158.005 67.4225) (end 159.1325 68.55) (width 0.5) (layer "B.Cu") (net 5))
   (segment (start 182.1 88.36) (end 182.1 83.78) (width 0.5) (layer "B.Cu") (net 5))
-  (segment (start 147.175 62.59) (end 148.71 62.59) (width 0.5) (layer "B.Cu") (net 5))
   (segment (start 147.85 119.04) (end 162.4 133.59) (width 0.5) (layer "B.Cu") (net 5))
   (segment (start 128.06 102.2) (end 129.81 103.95) (width 0.5) (layer "B.Cu") (net 5))
@@
   (segment (start 142.99 58.78) (end 144.73 60.52) (width 0.25) (layer "B.Cu") (net 5))
   (segment (start 131.825 76.6) (end 120.965 76.6) (width 0.5) (layer "B.Cu") (net 5))
-  (segment (start 148.71 62.59) (end 150.65 64.53) (width 0.5) (layer "B.Cu") (net 5))
   (segment (start 178.825 78.65) (end 182.08 78.65) (width 0.5) (layer "B.Cu") (net 5))
   (segment (start 182.1 83.78) (end 182.1 84.38) (width 0.5) (layer "B.Cu") (net 5))
@@
   (segment (start 162.985 90.73) (end 148.155 105.56) (width 0.25) (layer "B.Cu") (net 12))
   (segment (start 165.47 90.73) (end 162.985 90.73) (width 0.25) (layer "B.Cu") (net 12))
+  (segment (start 142 114) (end 142.055 113.945) (width 0.25) (layer "F.Cu") (net 13))
+  (segment (start 139.5 114) (end 142 114) (width 0.25) (layer "F.Cu") (net 13))
   (segment (start 115.2 95.54) (end 123.65 95.54) (width 0.25) (layer "F.Cu") (net 13))
-  (segment (start 123.65 95.54) (end 147.81 119.7) (width 0.25) (layer "F.Cu") (net 13))
   (segment (start 147.81 119.7) (end 153.555 119.7) (width 0.25) (layer "F.Cu") (net 13))
+  (segment (start 134.805 106.695) (end 134.805 109.305) (width 0.25) (layer "F.Cu") (net 13))
+  (segment (start 134.805 109.305) (end 139.5 114) (width 0.25) (layer "F.Cu") (net 13))
+  (segment (start 123.65 95.54) (end 134.805 106.695) (width 0.25) (layer "F.Cu") (net 13))
+  (segment (start 142.055 113.945) (end 147.81 119.7) (width 0.25) (layer "F.Cu") (net 13))
   (via (at 115.2 95.54) (size 0.8) (drill 0.4) (layers "F.Cu" "B.Cu") (net 13))
   (segment (start 116.9 94.06) (end 116.68 94.06) (width 0.25) (layer "B.Cu") (net 13))
@@
   (segment (start 128.04 66.7) (end 130.01 68.67) (width 0.5) (layer "B.Cu") (net 47))
   (segment (start 126.1625 66.7) (end 128.04 66.7) (width 0.5) (layer "B.Cu") (net 47))
+  (segment (start 150.65 59.85) (end 150.59 59.79) (width 0.5) (layer "F.Cu") (net 49))
   (segment (start 154.54 63.74) (end 150.59 59.79) (width 0.5) (layer "B.Cu") (net 49))
   (segment (start 157.3075 68.55) (end 154.54 65.7825) (width 0.5) (layer "B.Cu") (net 49))
